File: kicad/clock.sch (KiCad schematic (older format))
At the start: 82 parts, among them J1 USB-SS-52100-001, Q1 PN2222A, SW1 HOUR, SW2 MIN, SW3 TIME, U1 74HC4060, U10 74HC390, U11 NE555P, U12 74HC4511, U13 74HC4511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

Commit message: Update clock.sch
Parts:
- U11: symbol dk_Clock-Timing-Programmable-Timers-and-Oscillators:NE555P -> clock-rescue:NE555P-dk_Clock-Timing-Programmable-Timers-and-Oscillators
- U5: symbol dk_Logic-Flip-Flops:SN74HC74N -> clock-rescue:SN74HC74N-dk_Logic-Flip-Flops
- XTAL1: symbol dk_Crystals:ECS-_327-12_5-34B-TR -> clock-rescue:ECS-_327-12_5-34B-TR-dk_Crystals
Changed lines of the file:
@@
 EESchema Schematic File Version 4
-LIBS:clock-cache
-EELAYER 29 0
+EELAYER 30 0
 EELAYER END
 $Descr A3 11693 16535 portrait
@@
 $EndComp
 $Comp
-L dk_Crystals:ECS-_327-12_5-34B-TR XTAL1
+L clock-rescue:ECS-_327-12_5-34B-TR-dk_Crystals XTAL1
 U 1 1 5D03E855
 P 1300 1650
@@
 $EndComp
 $Comp
-L dk_Logic-Flip-Flops:SN74HC74N U5
+L clock-rescue:SN74HC74N-dk_Logic-Flip-Flops U5
 U 1 1 5D03F41F
 P 4000 1750
@@
 $EndComp
 $Comp
-L dk_Clock-Timing-Programmable-Timers-and-Oscillators:NE555P U11
+L clock-rescue:NE555P-dk_Clock-Timing-Programmable-Timers-and-Oscillators U11
 U 1 1 5D95E044
 P 5750 11250
